Commit message: add realsense and octomap

File: src/drone_essentials/urdf/fixed_joint.urdf (robot description, URDF)
Before this commit: robot drone_fixed_joint, 5 links, 4 joints
Links:
- removed link elp_left_optical_frame
- removed link elp_right_optical_frame
Joints:
- removed joint elp_left_link
- removed joint elp_right_link
- removed joint r200_link
- added joint realsense_link: type fixed, parent base_link, child camera_link, origin xyz=0.1 0.0 -0.1 rpy=0.0 0.0 0.0
