Commit message: edit add models

File: src/drone_essentials/urdf/iris_model.xacro (robot description, xacro)
@@ -1,4 +1,5 @@
+<!-- DO NOT EDIT: Generated from iris.sdf.jinja -->
 <?xml version="1.0"?>
-<robot name="drone_fixed_joint">
+<robot name='iris'>
     <material name = "dark_gray">
       <color rgba = "0.3 0.3 0.3 1"/>
@@ -21,8 +22,8 @@
           <mesh filename= "file:///home/pc208/drone_ws/src/drone_essentials/meshes/iris_prop_cw.dae"/>
         </geometry>
-        <origin xyz="0.13 -0.22 0.023"/>
         <material name = "blue" />
       </visual>
     </link>
+<!-- "0.13 -0.22 0.023" -->
     <joint name="rotor_0_joint" type="fixed">
         <parent link = "base_link"/>
@@ -35,5 +36,4 @@
           <mesh filename= "file:///home/pc208/drone_ws/src/drone_essentials/meshes/iris_prop_cw.dae"/>
         </geometry>
-        <origin xyz="-0.13 0.2 0.023"/>
         <material name = "blue" />
       </visual>
@@ -49,5 +49,4 @@
           <mesh filename= "file:///home/pc208/drone_ws/src/drone_essentials/meshes/iris_prop_ccw.dae"/>
         </geometry>
-        <origin xyz="0.13 0.22 0.023"/>
         <material name = "blue" />
       </visual>
@@ -63,5 +62,4 @@
           <mesh filename= "file:///home/pc208/drone_ws/src/drone_essentials/meshes/iris_prop_ccw.dae"/>
         </geometry>
-        <origin xyz="-0.13 -0.2 0.023"/>
         <material name = "blue" />
       </visual>
@@ -77,5 +75,5 @@
       <parent link="base_link"/>
       <child link="laser"/>
-      <origin xyz="0.0 0.0 0.055" rpy="0 0 0"/>
+      <origin xyz="0.0 0.0 0.1" rpy="0 0 0"/>
     </joint>
     <link name="r200" />
@@ -83,5 +81,5 @@
       <parent link="base_link"/>
       <child link="r200"/>
-      <origin xyz="0.1 0.0 0.0" rpy="-1.57 0.0 -1.57"/>
+      <origin xyz="0.1 0.0 0.0" rpy="-1.57 0 -1.57"/>
     </joint>
 </robot>

Commit message: add rviz config

File: src/drone_essentials/urdf/iris_model.xacro (robot description, xacro)
@@ -12,5 +12,5 @@
       <visual>
         <geometry>
-            <mesh filename= "file:///home/pc208/drone_ws/src/drone_essentials/meshes/iris.stl"/>
+            <mesh filename= "file:///home/leekaidel/drone_ws/src/drone_essentials/meshes/iris.stl"/>
         </geometry>
         <material name = "dark_gray" />
@@ -20,5 +20,5 @@
       <visual name="rotor_0_visual">
         <geometry>
-          <mesh filename= "file:///home/pc208/drone_ws/src/drone_essentials/meshes/iris_prop_cw.dae"/>
+          <mesh filename= "file:///home/leekaidel/drone_ws/src/drone_essentials/meshes/iris_prop_cw.dae"/>
         </geometry>
         <material name = "blue" />
@@ -34,5 +34,5 @@
       <visual name="rotor_1_visual">
         <geometry>
-          <mesh filename= "file:///home/pc208/drone_ws/src/drone_essentials/meshes/iris_prop_cw.dae"/>
+          <mesh filename= "file:///home/leekaidel/drone_ws/src/drone_essentials/meshes/iris_prop_cw.dae"/>
         </geometry>
         <material name = "blue" />
@@ -47,5 +47,5 @@
       <visual name="rotor_2_visual">
         <geometry>
-          <mesh filename= "file:///home/pc208/drone_ws/src/drone_essentials/meshes/iris_prop_ccw.dae"/>
+          <mesh filename= "file:///home/leekaidel/drone_ws/src/drone_essentials/meshes/iris_prop_ccw.dae"/>
         </geometry>
         <material name = "blue" />
@@ -60,5 +60,5 @@
       <visual name="rotor_3_visual">
         <geometry>
-          <mesh filename= "file:///home/pc208/drone_ws/src/drone_essentials/meshes/iris_prop_ccw.dae"/>
+          <mesh filename= "file:///home/leekaidel/drone_ws/src/drone_essentials/meshes/iris_prop_ccw.dae"/>
         </geometry>
         <material name = "blue" />

Commit message: fix cartographergit statusgit status

File: src/drone_essentials/urdf/iris_model.xacro (robot description, xacro)
@@ -1,5 +1,5 @@
 <!-- DO NOT EDIT: Generated from iris.sdf.jinja -->
 <?xml version="1.0"?>
-<robot name='iris'>
+<robot name='drone_fixed_joint'>
     <material name = "dark_gray">
       <color rgba = "0.3 0.3 0.3 1"/>
@@ -8,4 +8,13 @@
       <color rgba="0 0 1 1"/>
     </material>
+   <!-- iris model -->
+    <!-- <link name="drone">
+      <visual>
+        <geometry>
+            <mesh filename= "file:///home/leekaidel/drone_ws/src/drone_essentials/meshes/iris.stl"/>
+        </geometry>
+        <material name = "dark_gray" />
+      </visual>
+    </link> -->
     <!-- iris model -->
     <link name="base_link">

Commit message: fix

File: src/drone_essentials/urdf/iris_model.xacro (robot description, xacro)
@@ -21,5 +21,5 @@
       <visual>
         <geometry>
-            <mesh filename= "file:///home/leekaidel/drone_ws/src/drone_essentials/meshes/iris.stl"/>
+            <mesh filename= "file:///home/leekai/drone_ws/src/drone_essentials/meshes/iris.stl"/>
         </geometry>
         <material name = "dark_gray" />
@@ -29,5 +29,5 @@
       <visual name="rotor_0_visual">
         <geometry>
-          <mesh filename= "file:///home/leekaidel/drone_ws/src/drone_essentials/meshes/iris_prop_cw.dae"/>
+          <mesh filename= "file:///home/leekai/drone_ws/src/drone_essentials/meshes/iris_prop_cw.dae"/>
         </geometry>
         <material name = "blue" />
@@ -43,5 +43,5 @@
       <visual name="rotor_1_visual">
         <geometry>
-          <mesh filename= "file:///home/leekaidel/drone_ws/src/drone_essentials/meshes/iris_prop_cw.dae"/>
+          <mesh filename= "file:///home/leekai/drone_ws/src/drone_essentials/meshes/iris_prop_cw.dae"/>
         </geometry>
         <material name = "blue" />
@@ -56,5 +56,5 @@
       <visual name="rotor_2_visual">
         <geometry>
-          <mesh filename= "file:///home/leekaidel/drone_ws/src/drone_essentials/meshes/iris_prop_ccw.dae"/>
+          <mesh filename= "file:///home/leekai/drone_ws/src/drone_essentials/meshes/iris_prop_ccw.dae"/>
         </geometry>
         <material name = "blue" />
@@ -69,5 +69,5 @@
       <visual name="rotor_3_visual">
         <geometry>
-          <mesh filename= "file:///home/leekaidel/drone_ws/src/drone_essentials/meshes/iris_prop_ccw.dae"/>
+          <mesh filename= "file:///home/leekai/drone_ws/src/drone_essentials/meshes/iris_prop_ccw.dae"/>
         </geometry>
         <material name = "blue" />

Commit message: fix drone params

File: src/drone_essentials/urdf/iris_model.xacro (robot description, xacro)
@@ -21,5 +21,5 @@
       <visual>
         <geometry>
-            <mesh filename= "file:///home/leekai/drone_ws/src/drone_essentials/meshes/iris.stl"/>
+            <mesh filename= "file:///home/leekaidel/drone_ws/src/drone_essentials/meshes/iris.stl"/>
         </geometry>
         <material name = "dark_gray" />
@@ -29,5 +29,5 @@
       <visual name="rotor_0_visual">
         <geometry>
-          <mesh filename= "file:///home/leekai/drone_ws/src/drone_essentials/meshes/iris_prop_cw.dae"/>
+          <mesh filename= "file:///home/leekaidel/drone_ws/src/drone_essentials/meshes/iris_prop_cw.dae"/>
         </geometry>
         <material name = "blue" />
@@ -43,5 +43,5 @@
       <visual name="rotor_1_visual">
         <geometry>
-          <mesh filename= "file:///home/leekai/drone_ws/src/drone_essentials/meshes/iris_prop_cw.dae"/>
+          <mesh filename= "file:///home/leekaidel/drone_ws/src/drone_essentials/meshes/iris_prop_cw.dae"/>
         </geometry>
         <material name = "blue" />
@@ -56,5 +56,5 @@
       <visual name="rotor_2_visual">
         <geometry>
-          <mesh filename= "file:///home/leekai/drone_ws/src/drone_essentials/meshes/iris_prop_ccw.dae"/>
+          <mesh filename= "file:///home/leekaidel/drone_ws/src/drone_essentials/meshes/iris_prop_ccw.dae"/>
         </geometry>
         <material name = "blue" />
@@ -69,5 +69,5 @@
       <visual name="rotor_3_visual">
         <geometry>
-          <mesh filename= "file:///home/leekai/drone_ws/src/drone_essentials/meshes/iris_prop_ccw.dae"/>
+          <mesh filename= "file:///home/leekaidel/drone_ws/src/drone_essentials/meshes/iris_prop_ccw.dae"/>
         </geometry>
         <material name = "blue" />
